File: no-vga-freetracing/justin-freetracing.kicad_pcb (KiCad board)
At the start: 2 copper layers, 237.6 x 136.2 mm, 129 parts, among them J1 DB15_Female_HighDensity, J2 Conn_02x03_Odd_Even, J3 Conn_01x08_MountingPin, J5 Barrel_Jack_Switch_Pin3Ring, K1 SW_Push, K10 SW_Push, K11 SW_Push, K12 SW_Push, K13 SW_Push, K14 SW_Push, K15 SW_Push, K16 SW_Push, K17 SW_Push, K18 SW_Push, K19 SW_Push, K2 SW_Push, K20 SW_Push, K21 SW_Push, K22 SW_Push, K23 SW_Push, K24 SW_Push, K25 SW_Push, K26 SW_Push, K27 SW_Push, K28 SW_Push, K29 SW_Push, K3 SW_Push, K30 SW_Push, K31 SW_Push, K32 SW_Push, K33 SW_Push, K34 SW_Push, K35 SW_Push, K36 SW_Push, K37 SW_Push, K38 SW_Push, K39 SW_Push, K4 SW_Push, K40 SW_Push, K41 SW_Push, K42 SW_Push, K43 SW_Push, K44 SW_Push, K45 SW_Push, K46 SW_Push, K47 SW_Push, K48 SW_Push, K49 SW_Push, K5 SW_Push, K6 SW_Push, K7 SW_Push, K8 SW_Push, K9 SW_Push, U1 ATmega1284-P, Y1 20MHz

Commit message: Additional
Parts:
- removed R49, R50, R51: 1.5k, Resistor_THT:R_Axial_DIN0204_L3.6mm_D1.6mm_P5.08mm_Horizontal
- removed R52, R53, R54: 680, Resistor_THT:R_Axial_DIN0204_L3.6mm_D1.6mm_P5.08mm_Horizontal
- added U2: ICE40UL1K-SWG16, Package_CSP:WLCSP-16_1.409x1.409mm_P0.35mm, F.Cu at (46.8, 91.4)
- J1: value DB15_Female_HighDensity -> Conn_01x08_MountingPin; footprint Connector_Dsub:DSUB-15_Female_Horizontal_P2.77x2.54mm_EdgePinOffset9.40mm -> Connector_PinHeader_2.54mm:PinHeader_1x08_P2.54mm_Vertical
- moved J1 24.6 mm to (54.9, 64.0), turned to -90 degrees
- moved C4 5.79 mm to (57.1, 57.4)
Connections:
- J1 pad 1: /RED -> Net-(U1-Pad14)
- J1 pad 2: /GREEN -> Net-(U1-Pad15)
- J1 pad 3: /BLUE -> Net-(U1-Pad16)
- J1 pad 4: unconnected-(J1-Pad4) -> Net-(U1-Pad17)
- J1 pad 5: GND -> Net-(U1-Pad18)
- J1 pad 6: GND -> Net-(U1-Pad19)
- J1 pad 7: GND -> Net-(U1-Pad20)
- J1 pad 8: GND -> Net-(U1-Pad21)
- U1 pad 14: Net-(R50-Pad2) -> Net-(U1-Pad14)
- U1 pad 15: Net-(R54-Pad2) -> Net-(U1-Pad15)
- U1 pad 16: Net-(R49-Pad2) -> Net-(U1-Pad16)
- U1 pad 17: Net-(R52-Pad2) -> Net-(U1-Pad17)
- U1 pad 18: Net-(R51-Pad2) -> Net-(U1-Pad18)
- U1 pad 19: Net-(R53-Pad2) -> Net-(U1-Pad19)
- U1 pad 20: /VSYNC -> Net-(U1-Pad20)
- U1 pad 21: /HSYNC -> Net-(U1-Pad21)
Routing:
- net GND: track 226.1 -> 169.3 mm
- net /HSYNC: track 44.3 -> 0.00 mm
- net Net-(R50-Pad2): track 29.2 -> 0.00 mm
- net /VSYNC: track 26.5 -> 0.00 mm
- net Net-(R54-Pad2): track 23.0 -> 0.00 mm
- net Net-(U1-Pad21): track 0.00 -> 21.1 mm
- net Net-(R49-Pad2): track 19.2 -> 0.00 mm
- net Net-(R52-Pad2): track 15.2 -> 0.00 mm
- net /BLUE: track 9.10 -> 0.00 mm
- net Net-(R53-Pad2): track 6.85 -> 0.00 mm
- net Net-(R51-Pad2): track 6.85 -> 0.00 mm
- net /GREEN: track 6.10 -> 0.00 mm
- net /RED: track 5.40 -> 0.00 mm
- net Net-(U1-Pad20): track 0.00 -> 4.77 mm
- net Net-(U1-Pad19): track 0.00 -> 4.77 mm
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Other:
- board text added: "1 x Atmega1284-PU 4 x 0.1 uF Capacitors 2 x 18 pF Capacitors 2 x Red LEDs 1 x 20 MHz Oscillator 48 x Diodes 3 x 680 Ohm Resistor 2 x 1x8 Pin Headers 3 x 1.5k Ohm Resistor 1 x Barrel Jack Mount 1 x 2x3 Pin Headers 1 x 1x5 Pin Headers 2 x 220 Ohm Resistors 48 x Cherry/Outemu Switches"
- board text added: "PD0"
- board text added: "PD1"
- board text added: "PD2"
- board text added: "PD3"
- board text added: "PD4"
- board text added: "PD5"
- board text added: "PD6"
- board text added: "PD7"
- board text removed: "1 x Atmega1284-PU 4 x 0.1 uF Capacitors 2 x 18 pF Capacitors 2 x Red LEDs 1 x 20 MHz Oscillator 48 x Diodes 3 x 680 Ohm Resistor 1 x VGA Horizontal Mount 3 x 1.5k Ohm Resistor 1 x Barrel Jack Mount 1 x 2x3 Pin Headers 1 x 1x5 Pin Headers 2 x 220 Ohm Resistors 48 x Cherry/Outemu Switches"
- board text removed: "HSYNC"
- board text removed: "RED"
- board text removed: "VSYNC"
